Commit message: Change in robot color and included with camera

File: urdf/macro.xacro (robot description, xacro)
@@ -22,7 +22,28 @@
         </link>
     </xacro:macro>
-    <xacro:macro name="joint_wheel" params="name child origin_xyz axis_xyz">
+       <xacro:macro name="link_dummy" params="name">
+        <link name="${name}">
+            <inertial>
+              <mass value="0.2"/>
+              <origin rpy="0 0 0" xyz="0 0 0"/>
+              <inertia ixx="0.000526666666667" ixy="0" ixz="0" iyy="0.000526666666667" iyz="0" izz="0.001"/>
+            </inertial>
+            <collision name="link_right_wheel_collision">
+              <origin rpy="0 0 1.5707" xyz="0.0 0 0"/>
+              <geometry>
+                <mesh filename="package://pmr/meshes/xbox.dae" scale="0.01 0.01 0.01"/>
+              </geometry>
+            </collision>
+            <visual name="${name}_visual">
+              <origin rpy="0 0 1.5707" xyz="0.0 0 0"/>
+              <geometry>
+                <mesh filename="package://pmr/meshes/xbox.dae" scale="0.1 0.1 0.1"/>
+              </geometry>
+            </visual>
+        </link>
+    </xacro:macro>
+    <xacro:macro name="joint_wheel" params="name child origin_xyz axis_xyz origin_rpy">
       <joint name="${name}" type="continuous">
-        <origin rpy="0 0 0" xyz="${origin_xyz}"/>
+        <origin rpy="${origin_rpy}" xyz="${origin_xyz}"/>
         <child link="${child}"/>
         <parent link="link_chassis"/>

File: urdf/pmr.xacro (robot description, xacro)
@@ -9,8 +9,9 @@
     <inertial>
       <mass value="5"/>
-      <origin rpy="0 0 0" xyz="0 0 0.1"/>
+      <origin rpy="0 0 0" xyz="0 0  0.1"/>
       <inertia ixx="0.0395416666667" ixy="0" ixz="0" iyy="0.106208333333" iyz="0" izz="0.106208333333"/>
     </inertial>
     <collision name="collision_chassis">
+      <origin rpy="0 0 1.5707" xyz="0 0 0"/>
       <geometry>
         <mesh filename="package://pmr/meshes/link_chassis.stl" scale="0.001 0.001 0.001"/>
@@ -24,49 +25,24 @@
       <material name="blue"/>
     </visual>
-    <!-- caster front
-    <collision name="caster_front_collision">
-      <origin rpy=" 0 0 0" xyz="0.35 0 -0.025"/>
+  </link>
+  <!-- Camera -->
+  <link name="camera_link">
+    <collision>
+      <origin xyz="0 0 0" rpy="0 0 0"/>
       <geometry>
-        <sphere radius="0.025"/>
+        <box size="0.1 0.1 0.05 "/>
       </geometry>
-      <surface>
-        <friction>
-          <ode>
-            <mu>0</mu>
-            <mu2>0</mu2>
-            <slip1>1.0</slip1>
-            <slip2>1.0</slip2>
-          </ode>
-        </friction>
-      </surface>
     </collision>
-    <visual name="caster_front_visual">
-      <origin rpy=" 0 0 0" xyz="0.2 0 -0.025"/>
+    <visual>
+      <origin xyz="0 0 0" rpy="0 0 0"/>
       <geometry>
-        <sphere radius="0.025"/>
+        <box size="0.0001 0.0001 0.005 "/>
       </geometry>
     </visual>
-    <collision name="caster_back_collision">
-      <origin rpy=" 0 0 0" xyz="-0.35 0 -0.025"/>
-      <geometry>
-        <sphere radius="0.025"/>
-      </geometry>
-      <surface>
-        <friction>
-          <ode>
-            <mu>0</mu>
-            <mu2>0</mu2>
-            <slip1>1.0</slip1>
-            <slip2>1.0</slip2>
-          </ode>
-        </friction>
-      </surface>
-    </collision>
-    <visual name="caster_front_visual">
-      <origin rpy=" 0 0 0" xyz="-0.2 0 -0.025"/>
-      <geometry>
-        <sphere radius="0.0225"/>
-      </geometry>
-    </visual> -->
+    <inertial>
+      <mass value="1e-5" />
+      <origin xyz="0 0 0" rpy="0 0 0"/>
+      <inertia ixx="1e-6" ixy="0" ixz="0" iyy="1e-6" iyz="0" izz="1e-6" />
+    </inertial>
   </link>
   <link name="castor_front_link">
@@ -110,7 +86,10 @@
 <xacro:link_wheel name="link_right_wheel" />
 <xacro:link_wheel name="link_left_wheel" />
-<xacro:joint_wheel name="joint_right_wheel"  child="link_right_wheel"  origin_xyz="0 0.2 0" axis_xyz="0 1 0" />
-<xacro:joint_wheel name="joint_left_wheel"   child="link_left_wheel"   origin_xyz="0 -0.2 0" axis_xyz="0 1 0" />
-<xacro:joint_wheel name="joint_castor_front"   child="castor_front_link"   origin_xyz="0.2 0 -0.025" axis_xyz="1 0 0" />
-<xacro:joint_wheel name="joint_castor_back"   child="castor_back_link"   origin_xyz="-0.2 0 -0.025" axis_xyz="1 0 0" />
+<xacro:link_dummy name="link_dummy" />
+<xacro:joint_wheel name="joint_right_wheel"  child="link_right_wheel"  origin_xyz="0 0.2 0" axis_xyz="0 1 0" origin_rpy="0 0 0"/>
+<xacro:joint_wheel name="joint_left_wheel"   child="link_left_wheel"   origin_xyz="0 -0.2 0" axis_xyz="0 1 0" origin_rpy="0 0 0"/>
+<xacro:joint_wheel name="joint_castor_front"   child="castor_front_link"   origin_xyz="0.2 0 -0.025" axis_xyz="1 0 0" origin_rpy="0 0 0"/>
+<xacro:joint_wheel name="joint_castor_back"   child="castor_back_link"   origin_xyz="-0.2 0 -0.025" axis_xyz="1 0 0" origin_rpy="0 0 0"/>
+<xacro:joint_wheel name="camera_joint"   child="camera_link"   origin_xyz="0 0 0.55" axis_xyz="0 1 0" origin_rpy="0 0 0"/>
+<xacro:joint_wheel name="dummy_joint"   child="link_dummy"   origin_xyz="0 0 0.44" axis_xyz="0 1 0" origin_rpy="0 0 0"/>
 </robot>

Commit message: HAR Model imported

File: urdf/macro.xacro (robot description, xacro)
@@ -22,25 +22,4 @@
         </link>
     </xacro:macro>
-       <xacro:macro name="link_dummy" params="name">
-        <link name="${name}">
-            <inertial>
-              <mass value="0.2"/>
-              <origin rpy="0 0 0" xyz="0 0 0"/>
-              <inertia ixx="0.000526666666667" ixy="0" ixz="0" iyy="0.000526666666667" iyz="0" izz="0.001"/>
-            </inertial>
-            <collision name="link_right_wheel_collision">
-              <origin rpy="0 0 1.5707" xyz="0.0 0 0"/>
-              <geometry>
-                <mesh filename="package://pmr/meshes/xbox.dae" scale="0.01 0.01 0.01"/>
-              </geometry>
-            </collision>
-            <visual name="${name}_visual">
-              <origin rpy="0 0 1.5707" xyz="0.0 0 0"/>
-              <geometry>
-                <mesh filename="package://pmr/meshes/xbox.dae" scale="0.1 0.1 0.1"/>
-              </geometry>
-            </visual>
-        </link>
-    </xacro:macro>
     <xacro:macro name="joint_wheel" params="name child origin_xyz axis_xyz origin_rpy">
       <joint name="${name}" type="continuous">
@@ -53,3 +32,10 @@
       </joint>
     </xacro:macro>
+    <xacro:macro name="fixed_joint" params="name child origin_xyz origin_rpy">
+      <joint name="${name}" type="fixed">
+        <origin rpy="${origin_rpy}" xyz="${origin_xyz}"/>
+        <child link="${child}"/>
+        <parent link="link_chassis"/>
+      </joint>
+    </xacro:macro>
 </robot>

File: urdf/materials.xacro (robot description, xacro)
@@ -14,5 +14,5 @@
   </material>
   <material name="orange">
-    <color rgba="1.0 0.423529411765 0.0392156862745 1.0"/>
+    <color rgba="1.0 0.423529411765 0.0392156862745 0.5"/>
   </material>
   <material name="brown">
@@ -25,3 +25,9 @@
     <color rgba="1.0 1.0 1.0 1.0"/>
   </material>
+  <material name="alu">
+    <color rgba="132 135 137 0.5"/>
+  </material>
+  <material name="darkblue">
+    <color rgba="41 86 143 1.0"/>
+  </material>
 </robot>

File: urdf/pmr.xacro (robot description, xacro)
@@ -15,5 +15,5 @@
       <origin rpy="0 0 1.5707" xyz="0 0 0"/>
       <geometry>
-        <mesh filename="package://pmr/meshes/link_chassis.stl" scale="0.001 0.001 0.001"/>
+        <mesh filename="package://pmr/meshes/base.dae" scale="0.001 0.001 0.001"/>
       </geometry>
     </collision>
@@ -21,5 +21,5 @@
       <origin rpy="0 0 1.5707" xyz="0 0 0"/>
       <geometry>
-        <mesh filename="package://pmr/meshes/link_chassis.stl" scale="0.001 0.001 0.001"/>
+        <mesh filename="package://pmr/meshes/base.dae" scale="1 1 1"/>
       </geometry>
       <material name="blue"/>
@@ -55,5 +55,5 @@
       <origin rpy="0 0 0" xyz="0 0 0" />
       <geometry>
-        <sphere radius="0.025"/>
+        <mesh filename="package://pmr/meshes/har_castor_ball.stl" scale="0.001 0.001 0.001"/>
       </geometry>
     </collision>
@@ -61,5 +61,5 @@
       <origin rpy="0 0 0" xyz="0 0 0"/>
       <geometry>
-        <sphere radius="0.025"/>
+        <mesh filename="package://pmr/meshes/har_castor_ball.stl" scale="0.001 0.001 0.001"/>
       </geometry>
     </visual>
@@ -74,5 +74,5 @@
       <origin rpy="0 0 0" xyz="0 0 0" />
       <geometry>
-        <sphere radius="0.025"/>
+        <mesh filename="package://pmr/meshes/har_castor_ball.stl" scale="0.001 0.001 0.001"/>
       </geometry>
     </collision>
@@ -80,5 +80,66 @@
       <origin rpy="0 0 0" xyz="0 0 0"/>
       <geometry>
-        <sphere radius="0.025"/>
+        <mesh filename="package://pmr/meshes/har_castor_ball.stl" scale="0.001 0.001 0.001"/>
+      </geometry>
+    </visual>
+  </link>
+  <link name="middle_link">
+    <inertial>
+      <mass value="1"/>
+      <origin rpy="0 0 0" xyz="0 0 0"/>
+      <inertia ixx="0.052666666" ixy="0" ixz="0" iyy="0.052666666" iyz="0" izz="0.001"/>
+    </inertial>
+    <collision name="middle_collision">
+      <origin rpy="0 0 0" xyz="0 0 0" />
+      <geometry>
+        <mesh filename="package://pmr/meshes/middle.dae" scale="0.001 0.001 0.001"/>
+      </geometry>
+    </collision>
+    <visual name="middle_visual">
+      <origin rpy="0 0 0" xyz="0 0 0"/>
+      <geometry>
+        <mesh filename="package://pmr/meshes/middle.dae" scale="1 1 1"/>
+      </geometry>
+    </visual>
+  </link>
+  <link name="medic_link">
+    <collision name="medic_collision">
+      <origin rpy="0 0 0" xyz="0 0 0" />
+      <geometry>
+        <mesh filename="package://pmr/meshes/medic.dae" scale="0.001 0.001 0.001"/>
+      </geometry>
+    </collision>
+    <visual name="medic_visual">
+      <origin rpy="0 0 0" xyz="0 0 0"/>
+      <geometry>
+        <mesh filename="package://pmr/meshes/medic.dae" scale="1 1 1"/>
+      </geometry>
+    </visual>
+  </link>
+  <link name="head_link">
+    <collision name="head_collision">
+      <origin rpy="0 0 0" xyz="0 0 0" />
+      <geometry>
+        <mesh filename="package://pmr/meshes/head.dae" scale="0.001 0.001 0.001"/>
+      </geometry>
+    </collision>
+    <visual name="head_visual">
+      <origin rpy="0 0 0" xyz="0 0 0"/>
+      <geometry>
+        <mesh filename="package://pmr/meshes/head.dae" scale="1 1 1"/>
+      </geometry>
+    </visual>
+  </link>
+  <link name="support_link">
+    <collision name="support_collision">
+      <origin rpy="0 0 0" xyz="0 0 0" />
+      <geometry>
+        <mesh filename="package://pmr/meshes/support.dae" scale="1 1 1"/>
+      </geometry>
+    </collision>
+    <visual name="support_visual">
+      <origin rpy="0 0 0" xyz="0 0 0"/>
+      <geometry>
+        <mesh filename="package://pmr/meshes/support.dae" scale="1 1 1"/>
       </geometry>
     </visual>
@@ -86,10 +147,12 @@
 <xacro:link_wheel name="link_right_wheel" />
 <xacro:link_wheel name="link_left_wheel" />
-<xacro:link_dummy name="link_dummy" />
-<xacro:joint_wheel name="joint_right_wheel"  child="link_right_wheel"  origin_xyz="0 0.2 0" axis_xyz="0 1 0" origin_rpy="0 0 0"/>
-<xacro:joint_wheel name="joint_left_wheel"   child="link_left_wheel"   origin_xyz="0 -0.2 0" axis_xyz="0 1 0" origin_rpy="0 0 0"/>
-<xacro:joint_wheel name="joint_castor_front"   child="castor_front_link"   origin_xyz="0.2 0 -0.025" axis_xyz="1 0 0" origin_rpy="0 0 0"/>
-<xacro:joint_wheel name="joint_castor_back"   child="castor_back_link"   origin_xyz="-0.2 0 -0.025" axis_xyz="1 0 0" origin_rpy="0 0 0"/>
-<xacro:joint_wheel name="camera_joint"   child="camera_link"   origin_xyz="0 0 0.55" axis_xyz="0 1 0" origin_rpy="0 0 0"/>
-<xacro:joint_wheel name="dummy_joint"   child="link_dummy"   origin_xyz="0 0 0.44" axis_xyz="0 1 0" origin_rpy="0 0 0"/>
+<xacro:joint_wheel name="joint_right_wheel"  child="link_right_wheel"  origin_xyz="-0.0 0.24 0.0325" axis_xyz="0 1 0" origin_rpy="0 0 0"/>
+<xacro:joint_wheel name="joint_left_wheel"   child="link_left_wheel"   origin_xyz="-0.0 -0.24 0.0325" axis_xyz="0 1 0" origin_rpy="0 0 0"/>
+<xacro:joint_wheel name="joint_castor_front"   child="castor_front_link"   origin_xyz="0.2 0 -0.0175" axis_xyz="0 0 1" origin_rpy="0 0 0"/>
+<xacro:joint_wheel name="joint_castor_back"   child="castor_back_link"   origin_xyz="-0.2 0 -0.0175" axis_xyz="0 0 1" origin_rpy="0 0 0"/>
+<xacro:joint_wheel name="camera_joint"   child="camera_link"   origin_xyz="0.25 0 1.5" axis_xyz="0 1 0" origin_rpy="0 0 0"/>
+<xacro:fixed_joint name="joint_middle"   child="middle_link"   origin_xyz="0 0 0" origin_rpy="0 0 1.5708"/>
+<xacro:fixed_joint name="joint_medic"   child="medic_link"   origin_xyz="0 0 0" origin_rpy="0 0 1.5708"/>
+<xacro:fixed_joint name="joint_head"   child="head_link"   origin_xyz="0 0 0" origin_rpy="0 0 1.5708"/>
+<xacro:fixed_joint name="joint_support"   child="support_link"   origin_xyz="0 0 0" origin_rpy="0 0 1.5708"/>
 </robot>
